File: bt-0801.kicad_sch (KiCad schematic)
At the start: 37 parts

Commit message: fix : add name.
Parts:
- gave numbers to parts that had none: 36
- renumbered ESP_DBG to ESP_DBG1

Commit message: altium_28
Parts:
- D201: renamed from D1; value DIODE -> SK34
- ESP_BOOT: renamed from SW1; value ESP_BOOT -> IT-110NHA
- ESP_DBG1: value Conn_01x05 -> SMW250-04
- ESP_RST: renamed from SW2; value Reset -> IT-110NHA
- PW: renamed from J2; value PW -> SMW250-02
- R201: renamed from R1; value R -> 2k
- R202: renamed from R2; value R -> 10k
- R203: renamed from R5; value R -> 10k
- SENSOR_1: renamed from J1; value SENSOR_1 -> 53047-0410
- SW101: renamed from SW4; value SW_DIP_x04 -> BSD-104
- SW201: renamed from SW3; value SW_SPDT -> 450301014042
- renumbered BT1 to BT201, BT2 to BT202, BT3 to BT203, BT4 to BT204, C6 to C101, C5 to C102, C4 to C103, C1 to C201, C2 to C202, C3 to C203, D2 to D101, L1 to L201, Q1 to Q201, Q2 to Q202, R8 to R101, R13 to R102, R12 to R103, R11 to R104, R6 to R105, R7 to R106, R9 to R107, R10 to R108, R3 to R204, R4 to R205, U2 to U101, U1 to U201
Other:
- moved on the sheet: R105, R106, R108
