File: bt-0808/bt-0801.kicad_pcb (KiCad board)
At the start: 2 copper layers, 120 x 120 mm, 37 parts, among them J2 PW, Q1 MMBT3904, Q2 IRLML6402, SW4 SW_DIP_x04, U101 ESP32-WROOM-32U, U201 TPS63030DSK

Commit message: pcb_update
Routing:
- net /BOOT: track 6.02 -> 19.2 mm
Changed lines of the file:
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@@
   (segment (start 112.5775 132.76) (end 112.5875 132.75) (width 0.25) (layer "F.Cu") (net 22))
   (segment (start 116.055 42.755) (end 116.055 111.695) (width 0.25) (layer "F.Cu") (net 22))
+  (segment (start 129 41.755) (end 137.745 41.755) (width 0.25) (layer "F.Cu") (net 31))
   (segment (start 139.29 37.94) (end 139.35 38) (width 0.25) (layer "F.Cu") (net 31))
+  (segment (start 137.745 41.755) (end 139.35 40.15) (width 0.25) (layer "F.Cu") (net 31))
   (segment (start 139.29 32) (end 139.29 37.94) (width 0.25) (layer "F.Cu") (net 31))
+  (segment (start 139.35 40.15) (end 139.35 38) (width 0.25) (layer "F.Cu") (net 31))
   (segment (start 142.695 30.325) (end 144.37 32) (width 0.25) (layer "F.Cu") (net 40))
   (segment (start 129 30.325) (end 142.695 30.325) (width 0.25) (layer "F.Cu") (net 40))

Commit message: test_new_line
Routing:
- net GND: track 187.4 -> 202.0 mm
Changed lines of the file:
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@@
   (segment (start 87.3 40.625) (end 87.175 40.75) (width 0.25) (layer "F.Cu") (net 5))
   (segment (start 122.005 25.245) (end 119.5 27.75) (width 0.25) (layer "F.Cu") (net 6))
+  (segment (start 149.76 38) (end 154.94 43.18) (width 0.25) (layer "F.Cu") (net 6))
   (segment (start 104.8 26.5) (end 104.8 28.75) (width 0.25) (layer "F.Cu") (net 6))
   (segment (start 129 25.245) (end 122.005 25.245) (width 0.25) (layer "F.Cu") (net 6))
@@
   (segment (start 141.83 32) (end 141.83 36.33) (width 0.25) (layer "F.Cu") (net 6))
   (segment (start 143.5 38) (end 147.15 38) (width 0.25) (layer "F.Cu") (net 6))
+  (segment (start 154.94 43.18) (end 154.75 43.37) (width 0.25) (layer "F.Cu") (net 6))
+  (segment (start 154.75 43.37) (end 154.75 47.75) (width 0.25) (layer "F.Cu") (net 6))
   (segment (start 104.8 25.95) (end 105.505 25.245) (width 0.25) (layer "F.Cu") (net 6))
   (segment (start 104.8 26.5) (end 104.8 25.95) (width 0.25) (layer "F.Cu") (net 6))
@@
   (segment (start 119.5 35) (end 119.5 32.745) (width 0.25) (layer "F.Cu") (net 6))
   (segment (start 112 25.245) (end 117.245 25.245) (width 0.25) (layer "F.Cu") (net 6))
+  (segment (start 147.15 38) (end 149.76 38) (width 0.25) (layer "F.Cu") (net 6))
   (segment (start 105.505 25.245) (end 112 25.245) (width 0.25) (layer "F.Cu") (net 6))
   (segment (start 141.83 36.33) (end 143.5 38) (width 0.25) (layer "F.Cu") (net 6))

Commit message: 각부품값수정
Routing:
- net GND: track 202.0 -> 187.4 mm
