File: bt-0808/bt-0801.kicad_sch (KiCad schematic)
At the start: 37 parts, among them J2 PW, Q1 MMBT3904, Q2 IRLML6402, SW4 SW_DIP_x04, U101 ESP32-WROOM-32U, U201 TPS63030DSK

Commit message: 각부품값수정
Parts:
- renumbered BT1 to BT201, BT2 to BT202, BT3 to BT203, BT4 to BT204, C6 to C101, C5 to C102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
